Commit message: [data] Add new tasks

File: raven/assets/hammer/kit.urdf (robot description, URDF)
Before this commit: robot kit.urdf, 1 links, 0 joints
Links:
- link baseLink: geometry collision box size=.28 .2 .005; visual box size=.28 .2 .005

File: raven/assets/plier/object-template.urdf (robot description, URDF)
Before this commit: robot object.urdf, 1 links, 0 joints
Links:
- link baseLink: geometry collision mesh filename=FNAMECOLL0 scale=SCALE0 SCALE1 SCALE2; visual mesh filename=FNAME0 scale=SCALE0 SCALE1 SCALE2

File: raven/assets/screwdriver/kit.urdf (robot description, URDF)
Before this commit: robot kit.urdf, 1 links, 0 joints
Links:
- link baseLink: geometry collision box size=0.24, 0.26, 0.005; visual box size=0.24, 0.26, 0.005

Commit message: [Task] 3D tool

File: raven/assets/hammer/kit.urdf (robot description, URDF)
Before this commit: robot kit.urdf, 1 links, 0 joints
Links:
- link baseLink: geometry collision box size=0.28, 0.26, 0.005; visual box size=0.28, 0.26, 0.005

File: raven/assets/screwdriver/kit.urdf (robot description, URDF)
Before this commit: robot kit.urdf, 1 links, 0 joints
Links:
- link baseLink: geometry collision box size=0.28, 0.26, 0.005; visual box size=0.28, 0.26, 0.005
